Commit message: Update URI paths and include hooks in wamv_gazebo

File: vrx_urdf/wamv_description/urdf/thrusters/engine.xacro (robot description, xacro)
@@ -6,5 +6,5 @@
       <visual>
         <geometry>
-          <mesh filename="package://wamv_description/models/engine/mesh/engine.dae"/>
+          <mesh filename="package://engine/mesh/engine.dae"/>
         </geometry>
       </visual>
@@ -29,5 +29,5 @@
       <visual>
         <geometry>
-          <mesh filename="package://wamv_description/models/propeller/mesh/propeller.dae"/>
+          <mesh filename="package://propeller/mesh/propeller.dae"/>
         </geometry>
       </visual>

File: vrx_urdf/wamv_description/urdf/wamv_base.urdf.xacro (robot description, xacro)
@@ -84,9 +84,17 @@
     </collision>
   </xacro:macro>
+    <!-- Dummy base link for KDL support
+       KDL does not allow inertia on the base link -->
+    <link name="${namespace}/root_link"/>
+    <joint name="${namespace}/root_to_base" type="fixed">
+      <parent link="${namespace}/root_link"/>
+      <child link="${namespace}/base_link"/>
+      <origin xyz="0 0 0" rpy="0 0 0"/>
+    </joint>
   <!-- Basic model of the 16' WAM-V USV -->
   <link name="${namespace}/base_link">
     <visual>
       <geometry>
-        <mesh filename="package://wamv_description/models/WAM-V-Base/mesh/WAM-V-Base.dae"/>
+        <mesh filename="package://WAM-V-Base/mesh/WAM-V-Base.dae"/>
       </geometry>
     </visual>
@@ -118,8 +126,8 @@
         <pbr>
           <metal>
-            <albedo_map>model://wamv_description/models/WAM-V-Base/mesh/WAM-V_Albedo.png</albedo_map>
-            <normal_map>model://wamv_description/models/WAM-V-Base/mesh/WAM-V_Normal.png</normal_map>
-            <roughness_map>model://wamv_description/models/WAM-V-Base/mesh/WAM-V_Roughness.png</roughness_map>
-            <metalness_map>model://wamv_description/models/WAM-V-Base/mesh/WAM-V_Metalness.png</metalness_map>
+            <albedo_map>model://WAM-V-Base/mesh/WAM-V_Albedo.png</albedo_map>
+            <normal_map>model://WAM-V-Base/mesh/WAM-V_Normal.png</normal_map>
+            <roughness_map>model://WAM-V-Base/mesh/WAM-V_Roughness.png</roughness_map>
+            <metalness_map>model://WAM-V-Base/mesh/WAM-V_Metalness.png</metalness_map>
           </metal>
         </pbr>

File: vrx_urdf/wamv_gazebo/urdf/components/wamv_gps.xacro (robot description, xacro)
@@ -6,5 +6,5 @@
       <visual name="${name}_visual">
         <geometry>
-          <mesh filename="package://wamv_gazebo/models/gps/mesh/gps.dae"/>
+          <mesh filename="model://gps/mesh/gps.dae"/>
         </geometry>
       </visual>
